Commit message: Modelos entrenados con la camara apuntando hacia abajo

File: ros/src/robots/robotino/robotino_description/urdf/robotino.xacro (robot description, xacro)
@@ -174,10 +174,10 @@
       <inertia ixx="1.0" ixy="0.0" ixz="0.0" iyy="1.0" iyz="0.0" izz="1.0"/>
     </inertial>
-    <visual>
+    <!-- <visual>
       <origin rpy="0 0 1.570795" xyz="0 0 -0.06"/>
       <geometry>
         <mesh filename="package://robotino_description/meshes/RobotinoLaserScanner.dae" scale="0.01 0.01 0.01"/>
       </geometry>
-    </visual>
+    </visual> -->
     <collision>
       <origin rpy="0 0 1.570795" xyz="0 0 -0.06"/>
@@ -213,5 +213,5 @@
   </link>
   <joint name="camera_joint" type="fixed">
-    <origin rpy="0 0 0" xyz="0.1 0 0.2"/>
+    <origin rpy="0 0.9 0" xyz="0.1 0 0.2"/>
     <parent link="base_link"/>
     <child link="camera_link"/>
